File: Phase D/PCB_Design/Phase_D_STM_Shield/Phase_D_STM_Shield.kicad_pcb (KiCad board)
At the start: 2 copper layers, 76.8 x 85.1 mm, 6 parts, among them J1 Discovery Board Conn 1, J2 Discovery Board Conn 2

Commit message: Edits
Connections:
- MOTION_SENSOR1 pad 1: (no net) -> +5V
- MOTION_SENSOR1 pad 2: (no net) -> OUT
- MOTION_SENSOR1 pad 3: (no net) -> GND
Routing:
- net (no net): track 148.8 -> 0.00 mm, vias 6 -> 0
- net OUT: track 0.00 -> 57.9 mm, vias 0 -> 2
- net +5V: track 0.00 -> 50.6 mm, vias 0 -> 2
- net GND: track 50.3 -> 86.0 mm, vias 0 -> 2
Changed lines of the file:
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@@
     (fp_line (start 1.27 6.35) (end -1.27 6.35)
       (stroke (width 0.1) (type solid)) (layer "F.Fab"))
-    (pad "1" thru_hole rect (at 0 0 90) (size 1.7 1.7) (drill 1) (layers "*.Cu" "*.Mask"))
-    (pad "2" thru_hole oval (at 0 2.54 90) (size 1.7 1.7) (drill 1) (layers "*.Cu" "*.Mask"))
-    (pad "3" thru_hole oval (at 0 5.08 90) (size 1.7 1.7) (drill 1) (layers "*.Cu" "*.Mask"))
+    (pad "1" thru_hole rect (at 0 0 90) (size 1.7 1.7) (drill 1) (layers "*.Cu" "*.Mask")
+      (net 32 "+5V") (pinfunction "VCC") (pintype "input"))
+    (pad "2" thru_hole oval (at 0 2.54 90) (size 1.7 1.7) (drill 1) (layers "*.Cu" "*.Mask")
+      (net 75 "OUT") (pinfunction "OUT") (pintype "output"))
+    (pad "3" thru_hole oval (at 0 5.08 90) (size 1.7 1.7) (drill 1) (layers "*.Cu" "*.Mask")
+      (net 1 "GND") (pinfunction "GND") (pintype "input"))
     (model "${KICAD6_3DMODEL_DIR}/Connector_PinSocket_2.54mm.3dshapes/PinSocket_1x03_P2.54mm_Vertical.wrl"
       (offset (xyz 0 0 0))
@@
   (gr_rect (start 80.645 27.94) (end 157.48 113.03)
     (stroke (width 0.1) (type default)) (fill none) (layer "Edge.Cuts"))
-  (segment (start 88.36 53.435) (end 88.70415 53.77915) (width 0.25) (layer "F.Cu") (net 0))
-  (segment (start 87.0845 52.705) (end 87.8145 53.435) (width 0.25) (layer "F.Cu") (net 0))
-  (segment (start 109.855 35.56) (end 144.78 35.56) (width 0.25) (layer "F.Cu") (net 0))
-  (segment (start 145.32 43.91) (end 147.361701 43.91) (width 0.25) (layer "F.Cu") (net 0))
-  (segment (start 82.55 34.29) (end 82.55 52.705) (width 0.25) (layer "F.Cu") (net 0))
-  (segment (start 107.315 35.56) (end 102.87 31.115) (width 0.25) (layer "F.Cu") (net 0))
-  (segment (start 144.78 42.545) (end 148.05 42.545) (width 0.25) (layer "F.Cu") (net 0))
-  (segment (start 147.361701 43.91) (end 148.05 44.598299) (width 0.25) (layer "F.Cu") (net 0))
-  (segment (start 148.05 44.598299) (end 148.05 45.085) (width 0.25) (layer "F.Cu") (net 0))
-  (segment (start 144.145 45.085) (end 145.32 43.91) (width 0.25) (layer "F.Cu") (net 0))
-  (segment (start 130.175 43.18) (end 130.81 43.815) (width 0.25) (layer "F.Cu") (net 0))
-  (segment (start 87.8145 53.435) (end 88.36 53.435) (width 0.25) (layer "F.Cu") (net 0))
-  (segment (start 104.775 39.37) (end 108.585 43.18) (width 0.25) (layer "F.Cu") (net 0))
-  (segment (start 108.585 43.18) (end 130.175 43.18) (width 0.25) (layer "F.Cu") (net 0))
-  (segment (start 85.725 31.115) (end 82.55 34.29) (width 0.25) (layer "F.Cu") (net 0))
-  (segment (start 104.775 35.56) (end 104.775 39.37) (width 0.25) (layer "F.Cu") (net 0))
-  (segment (start 102.87 31.115) (end 85.725 31.115) (width 0.25) (layer "F.Cu") (net 0))
-  (via (at 87.0845 52.705) (size 0.8) (drill 0.4) (layers "F.Cu" "B.Cu") (net 0))
-  (via (at 144.78 35.56) (size 0.8) (drill 0.4) (layers "F.Cu" "B.Cu") (net 0))
-  (via (at 130.81 43.815) (size 0.8) (drill 0.4) (layers "F.Cu" "B.Cu") (net 0))
-  (via (at 144.145 45.085) (size 0.8) (drill 0.4) (layers "F.Cu" "B.Cu") (net 0))
-  (via (at 144.78 42.545) (size 0.8) (drill 0.4) (layers "F.Cu" "B.Cu") (net 0))
-  (via (at 82.55 52.705) (size 0.8) (drill 0.4) (layers "F.Cu" "B.Cu") (net 0))
-  (segment (start 144.78 35.56) (end 144.78 42.545) (width 0.25) (layer "B.Cu") (net 0))
-  (segment (start 130.81 43.815) (end 142.875 43.815) (width 0.25) (layer "B.Cu") (net 0))
-  (segment (start 142.875 43.815) (end 144.145 45.085) (width 0.25) (layer "B.Cu") (net 0))
-  (segment (start 82.55 52.705) (end 87.0845 52.705) (width 0.25) (layer "B.Cu") (net 0))
+  (segment (start 130.81 35.56) (end 133.985 38.735) (width 0.25) (layer "F.Cu") (net 1))
   (segment (start 133.745 62.9075) (end 133.745 55.065) (width 0.25) (layer "F.Cu") (net 1))
   (segment (start 133.745 55.065) (end 133.745 38.975) (width 0.25) (layer "F.Cu") (net 1))
+  (segment (start 144.78 42.545) (end 148.05 42.545) (width 0.25) (layer "F.Cu") (net 1))
+  (segment (start 133.745 38.975) (end 133.985 38.735) (width 0.25) (layer "F.Cu") (net 1))
+  (segment (start 109.855 35.56) (end 130.81 35.56) (width 0.25) (layer "F.Cu") (net 1))
   (segment (start 151.765 38.735) (end 151.765 42.545) (width 0.25) (layer "F.Cu") (net 1))
-  (segment (start 133.745 38.975) (end 133.985 38.735) (width 0.25) (layer "F.Cu") (net 1))
   (segment (start 133.985 38.735) (end 151.765 38.735) (width 0.25) (layer "F.Cu") (net 1))
   (segment (start 130.5725 66.08) (end 133.745 62.9075) (width 0.25) (layer "F.Cu") (net 1))
+  (via (at 144.78 35.56) (size 0.8) (drill 0.4) (layers "F.Cu" "B.Cu") (net 1))
+  (via (at 144.78 42.545) (size 0.8) (drill 0.4) (layers "F.Cu" "B.Cu") (net 1))
+  (segment (start 144.78 35.56) (end 144.78 42.545) (width 0.25) (layer "B.Cu") (net 1))
   (segment (start 86.36 107.95) (end 86.36 77.47) (width 0.25) (layer "F.Cu") (net 25))
   (segment (start 138.685 60.325) (end 142.24 60.325) (width 0.25) (layer "F.Cu") (net 25))
@@
   (segment (start 132.97 66.04) (end 138.685 60.325) (width 0.25) (layer "F.Cu") (net 25))
   (segment (start 142.24 78.105) (end 111.76 108.585) (width 0.25) (layer "F.Cu") (net 25))
+  (segment (start 144.145 45.085) (end 149.225 45.085) (width 0.25) (layer "F.Cu") (net 32))
+  (segment (start 104.775 39.37) (end 104.775 35.56) (width 0.25) (layer "F.Cu") (net 32))
+  (segment (start 130.175 43.18) (end 130.81 43.815) (width 0.25) (layer "F.Cu") (net 32))
+  (segment (start 104.775 39.37) (end 108.585 43.18) (width 0.25) (layer "F.Cu") (net 32))
+  (segment (start 108.585 43.18) (end 130.175 43.18) (width 0.25) (layer "F.Cu") (net 32))
+  (via (at 130.81 43.815) (size 0.8) (drill 0.4) (layers "F.Cu" "B.Cu") (net 32))
+  (via (at 144.145 45.085) (size 0.8) (drill 0.4) (layers "F.Cu" "B.Cu") (net 32))
+  (segment (start 130.81 43.815) (end 142.875 43.815) (width 0.25) (layer "B.Cu") (net 32))
+  (segment (start 142.875 43.815) (end 144.145 45.085) (width 0.25) (layer "B.Cu") (net 32))
   (segment (start 86.36 74.93) (end 89.535 74.93) (width 0.25) (layer "F.Cu") (net 73))
   (segment (start 107.315 49.53) (end 94.615 36.83) (width 0.25) (layer "F.Cu") (net 73))
@@
   (segment (start 131.445 70.485) (end 128.9975 68.0375) (width 0.25) (layer "F.Cu") (net 74))
   (segment (start 134.62 66.04) (end 131.445 69.215) (width 0.25) (layer "F.Cu") (net 74))
+  (segment (start 106.045 31.115) (end 107.315 32.385) (width 0.25) (layer "F.Cu") (net 75))
+  (segment (start 87.63 54.61) (end 89.535 54.61) (width 0.25) (layer "F.Cu") (net 75))
+  (segment (start 107.315 32.385) (end 107.315 35.56) (width 0.25) (layer "F.Cu") (net 75))
+  (segment (start 82.55 52.705) (end 82.55 34.29) (width 0.25) (layer "F.Cu") (net 75))
+  (segment (start 85.725 31.115) (end 106.045 31.115) (width 0.25) (layer "F.Cu") (net 75))
+  (segment (start 82.55 34.29) (end 85.725 31.115) (width 0.25) (layer "F.Cu") (net 75))
+  (segment (start 87.0845 52.705) (end 87.0845 55.1555) (width 0.25) (layer "F.Cu") (net 75))
+  (segment (start 87.0845 55.1555) (end 87.63 54.61) (width 0.25) (layer "F.Cu") (net 75))
+  (via (at 87.0845 52.705) (size 0.8) (drill 0.4) (layers "F.Cu" "B.Cu") (net 75))
+  (via (at 82.55 52.705) (size 0.8) (drill 0.4) (layers "F.Cu" "B.Cu") (net 75))
+  (segment (start 82.55 52.705) (end 87.0845 52.705) (width 0.25) (layer "B.Cu") (net 75))
 )
