File: Phase D/PCB_Design/Phase_D_STM_Shield/Phase_D_STM_Shield.kicad_sch (KiCad schematic)
At the start: 5 parts, among them J1 Discovery Board Conn 1, J2 Discovery Board Conn 2

Commit message: Hardware implementation of project
Parts:
- added MOTION_SENSOR1: ~, Connector_PinSocket_2.54mm:PinSocket_1x03_P2.54mm_Vertical, symbol Embedded:PIR_MOTION
- BZ1: renamed from BZ?; footprint (none) -> Buzzer_Beeper:MagneticBuzzer_PUI_AT-0927-TT-6-R
- D1: renamed from D?; footprint (none) -> LED_SMD:LED_0603_1608Metric
- R1: renamed from R?; footprint (none) -> Resistor_SMD:R_0603_1608Metric
Connections:
- net DS is gone; now on net GREEN_LED: J1.30 (Pin_30)
- net Dig4 is gone; now on net BUZZER: J1.28 (Pin_28)
- net +5V: now also MOTION_SENSOR1. (VCC)
- net GND: now also BZ1.2 (+), D1.2 (A), MOTION_SENSOR1. (VCC)
- net GREEN_LED: now also R1.1; no longer J1.40 (Pin_40)
- net at R1.2: now also D1.1 (K)
- net OUT: now reaches J1.12 (Pin_12)
- net OUT: now also MOTION_SENSOR1. (VCC)
- net BUZZER: now reaches BZ1.1 (-)
- net Button_1: no longer names the net of J1.44 (Pin_44)
- net Button_2: no longer names the net of J1.42 (Pin_42)
- net Buzzer: no longer names the net of J1.36 (Pin_36)
- net Dig1: no longer names the net of J1.20 (Pin_20)
- net Dig2: no longer names the net of J1.22 (Pin_22)
- net Dig3: no longer names the net of J1.26 (Pin_26)
- net INT: no longer names the net of J2.35 (Pin_35)
- net RED_LED: no longer names the net of J1.38 (Pin_38)
- net RX: no longer names the net of J1.13 (Pin_13)
- net SCL: no longer names the net of J2.24 (Pin_24)
- net SDA: no longer names the net of J2.23 (Pin_23)
- net SH_CP: no longer names the net of J1.34 (Pin_34)
- net ST_CP: no longer names the net of J1.32 (Pin_32)
- net TX: no longer names the net of J1.14 (Pin_14)
- no-connect marks 69 -> 83
Other:
- note added: "HRC-SR501 Motion Sensor"
- note added: "LED circuit"
- note added: "Piezo Buzzer"
- moved on the sheet: BZ1, D1, R1

Commit message: Edits
Connections:
- net +5V: now also MOTION_SENSOR1.1 (VCC); no longer MOTION_SENSOR1. (VCC)
- net GND: now also MOTION_SENSOR1.3 (GND); no longer MOTION_SENSOR1. (VCC)
- net OUT: now also MOTION_SENSOR1.2 (OUT); no longer MOTION_SENSOR1. (VCC)
Changed lines of the file:
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@@
+    (stroke (width 0) (type default))
+  )
+  (wire (pts (xy 190.5 45.72) (xy 190.5 44.45))
     (stroke (width 0) (type default))
   )
@@
     (stroke (width 0) (type default))
   )
+  (wire (pts (xy 186.69 45.72) (xy 186.69 44.45))
+    (stroke (width 0) (type default))
+  )
   (wire (pts (xy 69.85 27.94) (xy 73.66 27.94))
     (stroke (width 0) (type default))
@@
   )
   (wire (pts (xy 27.94 86.36) (xy 31.75 86.36))
+    (stroke (width 0) (type default))
+  )
+  (wire (pts (xy 194.31 45.72) (xy 194.31 44.45))
     (stroke (width 0) (type default))
   )
@@
     (effects (font (size 1.27 1.27) (thickness 0.254) bold) (justify left bottom))
   )
-  (global_label "OUT" (shape bidirectional) (at 190.5 44.45 270) (fields_autoplaced)
+  (global_label "OUT" (shape bidirectional) (at 190.5 45.72 270) (fields_autoplaced)
     (effects (font (size 1.27 1.27)) (justify right))
-    (property "Intersheetrefs" "${INTERSHEET_REFS}" (at 190.5 52.0957 90)
+    (property "Intersheetrefs" "${INTERSHEET_REFS}" (at 190.5 53.3657 90)
       (effects (font (size 1.27 1.27)) (justify right) hide)
     )
@@
     )
   )
-  (symbol (lib_id "power:GND") (at 194.31 44.45 0) (unit 1)
-    (in_bom yes) (on_board yes) (dnp no)
-    (property "Reference" "#PWR015" (at 194.31 50.8 0)
-      (effects (font (size 1.27 1.27)) hide)
-    )
-    (property "Value" "GND" (at 194.437 47.7012 90)
-      (effects (font (size 1.27 1.27)) (justify right))
-    )
-    (property "Footprint" "" (at 194.31 44.45 0)
-      (effects (font (size 1.27 1.27)) hide)
-    )
-    (property "Datasheet" "" (at 194.31 44.45 0)
+  (symbol (lib_id "power:GND") (at 194.31 45.72 0) (unit 1)
+    (in_bom yes) (on_board yes) (dnp no)
+    (property "Reference" "#PWR015" (at 194.31 52.07 0)
+      (effects (font (size 1.27 1.27)) hide)
+    )
+    (property "Value" "GND" (at 194.437 48.9712 90)
+      (effects (font (size 1.27 1.27)) (justify right))
+    )
+    (property "Footprint" "" (at 194.31 45.72 0)
+      (effects (font (size 1.27 1.27)) hide)
+    )
+    (property "Datasheet" "" (at 194.31 45.72 0)
       (effects (font (size 1.27 1.27)) hide)
     )
@@
     )
   )
-  (symbol (lib_id "power:+5V") (at 186.69 44.45 180) (unit 1)
-    (in_bom yes) (on_board yes) (dnp no)
-    (property "Reference" "#PWR014" (at 186.69 40.64 0)
-      (effects (font (size 1.27 1.27)) hide)
-    )
-    (property "Value" "+5V" (at 186.309 47.7012 90)
+  (symbol (lib_id "power:+5V") (at 186.69 45.72 180) (unit 1)
+    (in_bom yes) (on_board yes) (dnp no)
+    (property "Reference" "#PWR014" (at 186.69 41.91 0)
+      (effects (font (size 1.27 1.27)) hide)
+    )
+    (property "Value" "+5V" (at 186.309 48.9712 90)
       (effects (font (size 1.27 1.27)) (justify left))
     )
-    (property "Footprint" "" (at 186.69 44.45 0)
-      (effects (font (size 1.27 1.27)) hide)
-    )
-    (property "Datasheet" "" (at 186.69 44.45 0)
+    (property "Footprint" "" (at 186.69 45.72 0)
+      (effects (font (size 1.27 1.27)) hide)
+    )
+    (property "Datasheet" "" (at 186.69 45.72 0)
       (effects (font (size 1.27 1.27)) hide)
     )
@@
       (effects (font (size 1.27 1.27)) hide)
     )
-    (pin "")
-    (pin "")
-    (pin "")
-    (instances
-      (project "Phase_D_STM_Shield"
+    (pin "1")
+    (pin "2")
+    (pin "3")
+    (instances
+      (project "Phase_D_STM_Shield"
